Commit message: 修复gazebo中相机接口问题、删除部分无用文档

File: AstraDrone_ros1_ws/src/Swarm/astra_swarm_bringup/models/iris_mid360_d435.sdf.xacro (robot description, xacro)
@@ -12,4 +12,5 @@
   <xacro:arg name="robot_namespace" default="/uav1"/>
   <xacro:arg name="frame_prefix" default="uav1"/>
+  <xacro:arg name="gazebo_camera_name" default="UAV1_Camera"/>
   <xacro:arg name="camera_namespace" default="/uav1/d435"/>
   <xacro:arg name="lidar_namespace" default="/uav1/livox"/>
@@ -19,8 +20,10 @@
   <xacro:property name="robot_namespace" value="$(arg robot_namespace)"/>
   <xacro:property name="frame_prefix" value="$(arg frame_prefix)"/>
+  <xacro:property name="gazebo_camera_name"
+                  value="$(arg gazebo_camera_name)"/>
   <xacro:property name="camera_namespace" value="$(arg camera_namespace)"/>
   <xacro:property name="lidar_namespace" value="$(arg lidar_namespace)"/>
   <xacro:property name="d435_sensor_prefix"
-                  value="${frame_prefix}_d435_"/>
+                  value="${gazebo_camera_name}_"/>
   <model name="${model_name}">
     <include>
@@ -216,5 +219,5 @@
       <sensor name="${d435_sensor_prefix}color" type="camera">
         <pose>0.0325 0 0 3.14 -1.57 1.57</pose>
-        <camera name="color">
+        <camera name="${gazebo_camera_name}_color">
           <horizontal_fov>1.211</horizontal_fov>
           <image>
@@ -239,5 +242,5 @@
       <sensor name="${d435_sensor_prefix}ired1" type="camera">
         <pose>0.02 0 0 3.14 -1.57 1.57</pose>
-        <camera name="ired1">
+        <camera name="${gazebo_camera_name}_infra1">
           <horizontal_fov>1.571</horizontal_fov>
           <image>
@@ -262,5 +265,5 @@
       <sensor name="${d435_sensor_prefix}ired2" type="camera">
         <pose>-0.03 0 0 3.14 -1.57 1.57</pose>
-        <camera name="ired2">
+        <camera name="${gazebo_camera_name}_infra2">
           <horizontal_fov>1.571</horizontal_fov>
           <image>
@@ -285,5 +288,5 @@
       <sensor name="${d435_sensor_prefix}depth" type="depth">
         <pose>0.0325 0 0 3.14 -1.57 1.57</pose>
-        <camera name="depth">
+        <camera name="${gazebo_camera_name}_depth">
           <horizontal_fov>1.571</horizontal_fov>
           <image>
@@ -310,5 +313,5 @@
       <child>d435_link</child>
     </joint>
-    <plugin name="${frame_prefix}_d435"
+    <plugin name="${gazebo_camera_name}_plugin"
             filename="librealsense_gazebo_plugin.so">
       <prefix>${d435_sensor_prefix}</prefix>
